Commit message: 增加相机部分代码

File: src/cleaning_robot_description/urdf/cleaning_robot.urdf.xacro (robot description, xacro)
@@ -400,3 +400,69 @@
     </sensor>
   </gazebo>
+  <!-- 奥比中光深度相机 -->
+  <link name="orbbec_camera_link">
+    <visual>
+      <origin xyz="0 0 0" rpy="0 0 0"/>
+      <geometry>
+        <box size="0.03 0.09 0.025"/>
+      </geometry>
+      <material name="dark_grey">
+        <color rgba="0.3 0.3 0.3 1.0"/>
+      </material>
+    </visual>
+    <collision>
+      <origin xyz="0 0 0" rpy="0 0 0"/>
+      <geometry>
+        <box size="0.03 0.09 0.025"/>
+      </geometry>
+    </collision>
+    <inertial>
+      <origin xyz="0 0 0" rpy="0 0 0"/>
+      <mass value="0.15"/>
+      <inertia ixx="0.01" ixy="0.0" ixz="0.0" iyy="0.01" iyz="0.0" izz="0.01"/>
+    </inertial>
+  </link>
+  <joint name="orbbec_camera_joint" type="fixed">
+    <parent link="base_link"/>
+    <child link="orbbec_camera_link"/>
+    <origin xyz="0.20 0 0.20" rpy="0 0.2 0"/>
+  </joint>
+  <!-- Orbbec深度相机Gazebo插件 -->
+  <gazebo reference="orbbec_camera_link">
+    <sensor type="depth" name="orbbec_depth_sensor">
+      <update_rate>30.0</update_rate>
+      <camera name="orbbec_camera">
+        <horizontal_fov>1.047198</horizontal_fov>
+        <image>
+          <width>640</width>
+          <height>480</height>
+          <format>R8G8B8</format>
+        </image>
+        <clip>
+          <near>0.05</near>
+          <far>8.0</far>
+        </clip>
+        <noise>
+          <type>gaussian</type>
+          <mean>0.0</mean>
+          <stddev>0.007</stddev>
+        </noise>
+      </camera>
+      <plugin name="orbbec_depth_controller" filename="libgazebo_ros_depth_camera.so">
+        <ros>
+          <namespace>/cleaning_robot</namespace>
+          <remapping>image_raw:=orbbec_camera/color/image_raw</remapping>
+          <remapping>camera_info:=orbbec_camera/color/camera_info</remapping>
+          <remapping>depth/image_raw:=orbbec_camera/depth/image_raw</remapping>
+          <remapping>depth/camera_info:=orbbec_camera/depth/camera_info</remapping>
+          <remapping>points:=orbbec_camera/pointcloud</remapping>
+        </ros>
+        <camera_name>orbbec_camera</camera_name>
+        <frame_name>orbbec_camera_link</frame_name>
+        <hack_baseline>0.0</hack_baseline>
+        <min_depth>0.05</min_depth>
+        <max_depth>8.0</max_depth>
+      </plugin>
+    </sensor>
+  </gazebo>
 </robot>
